File: Hardware/Eagle/OSER0001_RFIDGadget_UnoShield/OSER_RFID_UnoShield.brd (EAGLE design)
At the start: 68.8 x 53.5 mm, 6 parts, among them U1 ARDUINOR3-BPLACE

Commit message: Changed to 5V for RFID Readers
Switched to the PN532 RFID reader which uses 5V.
Connections:
- net PWR_3V: no longer RFID_PWR.1
- net PWR_5V: now also RFID_PWR.1
Routing:
- net PWR_5V: track 50.2 -> 81.3 mm
- net PWR_3V: track 30.8 -> 0.00 mm
Changed lines of the file:
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@@
 <drawing>
 <settings>
-<setting alwaysvectorfont="yes"/>
+<setting alwaysvectorfont="no"/>
 <setting verticaltext="up"/>
 </settings>
@@
 <signal name="PWR_3V">
 <contactref element="U1" pad="3V"/>
-<contactref element="RFID_PWR" pad="1"/>
-<wire x1="8.382" y1="8.106" x2="32.28" y2="8.106" width="1.016" layer="1"/>
-<wire x1="32.28" y1="8.106" x2="35.56" y2="4.826" width="1.016" layer="1"/>
-<wire x1="35.56" y1="4.826" x2="35.56" y2="2.54" width="1.016" layer="1"/>
 </signal>
 <signal name="EXT_MASTER_RST">
@@
 <contactref element="U1" pad="5V"/>
 <contactref element="ACTUATORS" pad="4"/>
-<wire x1="38.1" y1="2.54" x2="38.1" y2="28.448" width="1.016" layer="1"/>
+<wire x1="38.1" y1="2.54" x2="38.1" y2="4.826" width="1.016" layer="1"/>
+<wire x1="38.1" y1="4.826" x2="38.1" y2="28.448" width="1.016" layer="1"/>
 <wire x1="38.1" y1="28.448" x2="47.752" y2="38.1" width="1.016" layer="1"/>
 <wire x1="47.752" y1="38.1" x2="58.364" y2="38.1" width="1.016" layer="1"/>
 <wire x1="58.364" y1="38.1" x2="58.42" y2="38.044" width="1.016" layer="1"/>
+<contactref element="RFID_PWR" pad="1"/>
+<wire x1="8.382" y1="8.106" x2="34.82" y2="8.106" width="1.016" layer="1"/>
+<wire x1="34.82" y1="8.106" x2="38.1" y2="4.826" width="1.016" layer="1"/>
 </signal>
 <signal name="CLOSED_LED">
